Commit message: xacro tags should be prepended with 'xacro' xml namespace.

File: kinova_description/urdf/j2n4s300_standalone.xacro (robot description, xacro)
@@ -37,5 +37,5 @@
     <origin xyz="0 0 0" rpy="0 0 0" />
   </joint>
-  <property name="robot_root" value="root" />
+  <xacro:property name="robot_root" value="root" />
   <xacro:j2n4s300  base_parent="${robot_root}"/>
 </robot>

File: kinova_description/urdf/j2n6s200_standalone.xacro (robot description, xacro)
@@ -37,5 +37,5 @@
     <origin xyz="0 0 0" rpy="0 0 0" />
   </joint>
-  <property name="robot_root" value="root" />
+  <xacro:property name="robot_root" value="root" />
   <xacro:j2n6s200  base_parent="${robot_root}"/>
 </robot>

File: kinova_description/urdf/j2n6s300_standalone.xacro (robot description, xacro)
@@ -37,5 +37,5 @@
     <origin xyz="0 0 0" rpy="0 0 0" />
   </joint>
-  <property name="robot_root" value="root" />
+  <xacro:property name="robot_root" value="root" />
   <xacro:j2n6s300  base_parent="${robot_root}"/>
 </robot>

File: kinova_description/urdf/j2n7s300_standalone.xacro (robot description, xacro)
@@ -37,5 +37,5 @@
     <origin xyz="0 0 0" rpy="0 0 0" />
   </joint>
-  <property name="robot_root" value="root" />
+  <xacro:property name="robot_root" value="root" />
   <xacro:j2n7s300  base_parent="${robot_root}"/>
 </robot>

File: kinova_description/urdf/j2s6s300_standalone.xacro (robot description, xacro)
@@ -37,5 +37,5 @@
     <origin xyz="0 0 0" rpy="0 0 0" />
   </joint>
-  <property name="robot_root" value="root" />
+  <xacro:property name="robot_root" value="root" />
   <xacro:j2s6s300  base_parent="${robot_root}"/>
 </robot>

File: kinova_description/urdf/j2s7s300_standalone.xacro (robot description, xacro)
@@ -37,5 +37,5 @@
     <origin xyz="0 0 0" rpy="0 0 0" />
   </joint>
-  <property name="robot_root" value="root" />
+  <xacro:property name="robot_root" value="root" />
   <xacro:j2s7s300  base_parent="${robot_root}"/>
 </robot>

File: kinova_description/urdf/kinova_common.xacro (robot description, xacro)
@@ -14,5 +14,5 @@
         xmlns:xacro="http://ros.org/wiki/xacro">
 <xacro:include filename="$(find kinova_description)/urdf/kinova_inertial.xacro" />
-    <property name="J_PI" value="3.1415926535897931" />
+    <xacro:property name="J_PI" value="3.1415926535897931" />
     <xacro:macro name="kinova_armlink" params="link_name link_mesh ring_mesh:=ring_big use_ring_mesh:=false mesh_no">
         <link name="${link_name}">

File: kinova_description/urdf/m1n4s200_standalone.xacro (robot description, xacro)
@@ -37,5 +37,5 @@
     <origin xyz="0 0 0" rpy="0 0 0" />
   </joint>
-  <property name="robot_root" value="root" />
+  <xacro:property name="robot_root" value="root" />
   <xacro:m1n4s200  base_parent="${robot_root}"/>
 </robot>

File: kinova_description/urdf/m1n6s200_standalone.xacro (robot description, xacro)
@@ -37,5 +37,5 @@
     <origin xyz="0 0 0" rpy="0 0 0" />
   </joint>
-  <property name="robot_root" value="root" />
+  <xacro:property name="robot_root" value="root" />
   <xacro:m1n6s200  base_parent="${robot_root}"/>
 </robot>

File: kinova_description/urdf/m1n6s300_standalone.xacro (robot description, xacro)
@@ -37,5 +37,5 @@
     <origin xyz="0 0 0" rpy="0 0 0" />
   </joint>
-  <property name="robot_root" value="root" />
+  <xacro:property name="robot_root" value="root" />
   <xacro:m1n6s300  base_parent="${robot_root}"/>
 </robot>
